File: Rele Module/Rele Module.sch (KiCad schematic (older format))
At the start: 9 parts, among them J1 Screw_Terminal_01x03, J2 Screw_Terminal_01x03, K1 DIPxx-1Cxx-51x, Q1 2N3904

Commit message: partially mapped footprints
Parts:
- D1: footprint (none) -> LED_SMD:LED_0805_2012Metric
- R1, R2, R3: footprint (none) -> Resistor_SMD:R_0805_2012Metric_Pad1.15x1.40mm_HandSolder
Changed lines of the file:
@@
 F 0 "R2" V 3293 3550 50  0000 C CNN
 F 1 "R" V 3384 3550 50  0000 C CNN
-F 2 "" V 3430 3550 50  0001 C CNN
+F 2 "Resistor_SMD:R_0805_2012Metric_Pad1.15x1.40mm_HandSolder" V 3430 3550 50  0001 C CNN
 F 3 "~" H 3500 3550 50  0001 C CNN
 	1    3500 3550
@@
 F 0 "R3" H 3920 3896 50  0000 L CNN
 F 1 "R" H 3920 3805 50  0000 L CNN
-F 2 "" V 3780 3850 50  0001 C CNN
+F 2 "Resistor_SMD:R_0805_2012Metric_Pad1.15x1.40mm_HandSolder" V 3780 3850 50  0001 C CNN
 F 3 "~" H 3850 3850 50  0001 C CNN
 	1    3850 3850
@@
 F 0 "R1" H 3220 3896 50  0000 L CNN
 F 1 "R" H 3220 3805 50  0000 L CNN
-F 2 "" V 3080 3850 50  0001 C CNN
+F 2 "Resistor_SMD:R_0805_2012Metric_Pad1.15x1.40mm_HandSolder" V 3080 3850 50  0001 C CNN
 F 3 "~" H 3150 3850 50  0001 C CNN
 	1    3150 3850
@@
 F 0 "D1" V 3189 4182 50  0000 R CNN
 F 1 "LED" V 3098 4182 50  0000 R CNN
-F 2 "" H 3150 4300 50  0001 C CNN
+F 2 "LED_SMD:LED_0805_2012Metric" H 3150 4300 50  0001 C CNN
 F 3 "~" H 3150 4300 50  0001 C CNN
 	1    3150 4300
