File: Rele Module/Rele Module.sch (KiCad schematic (older format))
At the start: 9 parts

Commit message: Main Commit
Parts:
- removed K?: DIPxx-1Cxx-51x, Relay_THT:Relay_StandexMeder_DIP_LowProfile, symbol Relay:DIPxx-1Cxx-51x
- added K1: SANYOU_SRD_Form_C, Relay_THT:Relay_SPDT_SANYOU_SRD_Series_Form_C, symbol Relay:SANYOU_SRD_Form_C
- D1: renamed from D?; footprint (none) -> LED_THT:LED_D5.0mm
- J1, J2: renamed from J?; footprint (none) -> TerminalBlock_Phoenix:TerminalBlock_Phoenix_MKDS-1,5-3-5.08_1x03_P5.08mm_Horizontal
- R1, R2, R3: renamed from R?; footprint (none) -> Resistor_THT:R_Axial_DIN0204_L3.6mm_D1.6mm_P7.62mm_Horizontal
- gave numbers to parts that had none: 2
Connections:
- net VCC: now also K1.5
- net at J2.1 (Pin_1): now also K1.4
- net at J2.2 (Pin_2): now also K1.3
- net at D2.2 (A), Q1.3 (C): now also K1.2
- net at J2.3 (Pin_3): now also K1.1
Changed lines of the file:
@@
 $EndDescr
 $Comp
-L Relay:DIPxx-1Cxx-51x K?
-U 1 1 5FB37991
-P 4700 2850
-F 0 "K?" H 5130 2896 50  0000 L CNN
-F 1 "DIPxx-1Cxx-51x" H 5130 2805 50  0000 L CNN
-F 2 "Relay_THT:Relay_StandexMeder_DIP_LowProfile" H 5150 2800 50  0001 L CNN
-F 3 "https://standexelectronics.com/wp-content/uploads/datasheet_reed_relay_DIP.pdf" H 4700 2850 50  0001 C CNN
-	1    4700 2850
-	1    0    0    -1
-$EndComp
-$Comp
-L Diode:1N4002 D?
+L Diode:1N4002 D2
 U 1 1 5FB38D03
 P 3850 2800
-F 0 "D?" V 3804 2880 50  0000 L CNN
+F 0 "D2" V 3804 2880 50  0000 L CNN
 F 1 "1N4002" V 3895 2880 50  0000 L CNN
 F 2 "Diode_THT:D_DO-41_SOD81_P10.16mm_Horizontal" H 3850 2625 50  0001 C CNN
@@
 $EndComp
 $Comp
-L Transistor_BJT:2N3904 Q?
+L Transistor_BJT:2N3904 Q1
 U 1 1 5FB3999D
 P 4400 3550
-F 0 "Q?" H 4590 3596 50  0000 L CNN
+F 0 "Q1" H 4590 3596 50  0000 L CNN
 F 1 "2N3904" H 4590 3505 50  0000 L CNN
 F 2 "Package_TO_SOT_THT:TO-92_Inline" H 4600 3475 50  0001 L CIN
@@
 $EndComp
 $Comp
-L Device:R R?
+L Device:R R2
 U 1 1 5FB3ACC1
 P 3500 3550
-F 0 "R?" V 3293 3550 50  0000 C CNN
+F 0 "R2" V 3293 3550 50  0000 C CNN
 F 1 "R" V 3384 3550 50  0000 C CNN
-F 2 "" V 3430 3550 50  0001 C CNN
+F 2 "Resistor_THT:R_Axial_DIN0204_L3.6mm_D1.6mm_P7.62mm_Horizontal" V 3430 3550 50  0001 C CNN
 F 3 "~" H 3500 3550 50  0001 C CNN
 	1    3500 3550
@@
 $EndComp
 $Comp
-L Device:R R?
+L Device:R R3
 U 1 1 5FB3B29B
 P 3850 3850
-F 0 "R?" H 3920 3896 50  0000 L CNN
+F 0 "R3" H 3920 3896 50  0000 L CNN
 F 1 "R" H 3920 3805 50  0000 L CNN
-F 2 "" V 3780 3850 50  0001 C CNN
+F 2 "Resistor_THT:R_Axial_DIN0204_L3.6mm_D1.6mm_P7.62mm_Horizontal" V 3780 3850 50  0001 C CNN
 F 3 "~" H 3850 3850 50  0001 C CNN
 	1    3850 3850
@@
 $EndComp
 $Comp
-L Device:R R?
+L Device:R R1
 U 1 1 5FB3B9DF
 P 3150 3850
-F 0 "R?" H 3220 3896 50  0000 L CNN
+F 0 "R1" H 3220 3896 50  0000 L CNN
 F 1 "R" H 3220 3805 50  0000 L CNN
-F 2 "" V 3080 3850 50  0001 C CNN
+F 2 "Resistor_THT:R_Axial_DIN0204_L3.6mm_D1.6mm_P7.62mm_Horizontal" V 3080 3850 50  0001 C CNN
 F 3 "~" H 3150 3850 50  0001 C CNN
 	1    3150 3850
@@
 $EndComp
 $Comp
-L Device:LED D?
+L Device:LED D1
 U 1 1 5FB3BCE4
 P 3150 4300
-F 0 "D?" V 3189 4182 50  0000 R CNN
+F 0 "D1" V 3189 4182 50  0000 R CNN
 F 1 "LED" V 3098 4182 50  0000 R CNN
-F 2 "" H 3150 4300 50  0001 C CNN
+F 2 "LED_THT:LED_D5.0mm" H 3150 4300 50  0001 C CNN
 F 3 "~" H 3150 4300 50  0001 C CNN
 	1    3150 4300
@@
 $EndComp
 $Comp
-L Connector:Screw_Terminal_01x03 J?
+L Connector:Screw_Terminal_01x03 J1
 U 1 1 5FB47837
 P 2750 2750
-F 0 "J?" H 2668 2425 50  0000 C CNN
+F 0 "J1" H 2668 2425 50  0000 C CNN
 F 1 "Screw_Terminal_01x03" H 2668 2516 50  0000 C CNN
-F 2 "" H 2750 2750 50  0001 C CNN
+F 2 "TerminalBlock_Phoenix:TerminalBlock_Phoenix_MKDS-1,5-3-5.08_1x03_P5.08mm_Horizontal" H 2750 2750 50  0001 C CNN
 F 3 "~" H 2750 2750 50  0001 C CNN
 	1    2750 2750
@@
 $EndComp
 $Comp
-L Connector:Screw_Terminal_01x03 J?
+L Connector:Screw_Terminal_01x03 J2
 U 1 1 5FB48265
 P 6200 2750
-F 0 "J?" H 6280 2792 50  0000 L CNN
+F 0 "J2" H 6280 2792 50  0000 L CNN
 F 1 "Screw_Terminal_01x03" H 6280 2701 50  0000 L CNN
-F 2 "" H 6200 2750 50  0001 C CNN
+F 2 "TerminalBlock_Phoenix:TerminalBlock_Phoenix_MKDS-1,5-3-5.08_1x03_P5.08mm_Horizontal" H 6200 2750 50  0001 C CNN
 F 3 "~" H 6200 2750 50  0001 C CNN
 	1    6200 2750
@@
 	5000 2450 5000 2550
 Wire Wire Line
-	6000 2850 5900 2850
-Wire Wire Line
-	5900 2850 5900 3200
-Wire Wire Line
-	5900 3200 4900 3200
+	6000 2850 5950 2850
+Wire Wire Line
+	5950 2850 5950 3200
+Wire Wire Line
+	5950 3200 4900 3200
 Wire Wire Line
 	4900 3200 4900 3150
@@
 	4500 2400 3850 2400
 $Comp
-L power:GND #PWR?
+L power:GND #PWR02
 U 1 1 5FB5713A
 P 3850 4750
-F 0 "#PWR?" H 3850 4500 50  0001 C CNN
+F 0 "#PWR02" H 3850 4500 50  0001 C CNN
 F 1 "GND" H 3855 4577 50  0000 C CNN
 F 2 "" H 3850 4750 50  0001 C CNN
@@
 $EndComp
 $Comp
-L power:VCC #PWR?
+L power:VCC #PWR01
 U 1 1 5FB579E1
 P 3850 2200
-F 0 "#PWR?" H 3850 2050 50  0001 C CNN
+F 0 "#PWR01" H 3850 2050 50  0001 C CNN
 F 1 "VCC" H 3865 2373 50  0000 C CNN
 F 2 "" H 3850 2200 50  0001 C CNN
@@
 Text Notes 7250 5050 2    50   ~ 0
 Rele Module
+$Comp
+L Relay:SANYOU_SRD_Form_C K1
+U 1 1 5FC4B47A
+P 4700 2850
+F 0 "K1" H 5130 2896 50  0000 L CNN
+F 1 "SANYOU_SRD_Form_C" H 5130 2805 50  0000 L CNN
+F 2 "Relay_THT:Relay_SPDT_SANYOU_SRD_Series_Form_C" H 5150 2800 50  0001 L CNN
+F 3 "http://www.sanyourelay.ca/public/products/pdf/SRD.pdf" H 4700 2850 50  0001 C CNN
+	1    4700 2850
+	1    0    0    -1
+$EndComp
 $EndSCHEMATC

Commit message: Make pcb connections
Connections:
- net at J2.1 (Pin_1): now also K1.3; no longer K1.4
- net at J2.2 (Pin_2): now also K1.1; no longer K1.3
- net at J2.3 (Pin_3): now also K1.4; no longer K1.1
Changed lines of the file:
@@
 Connection ~ 3850 4550
-Wire Wire Line
-	4800 2550 4800 2400
-Wire Wire Line
-	4800 2400 6000 2400
-Wire Wire Line
-	6000 2400 6000 2650
-Wire Wire Line
-	6000 2750 5900 2750
-Wire Wire Line
-	5900 2750 5900 2450
-Wire Wire Line
-	5900 2450 5000 2450
-Wire Wire Line
-	5000 2450 5000 2550
-Wire Wire Line
-	6000 2850 5950 2850
-Wire Wire Line
-	5950 2850 5950 3200
-Wire Wire Line
-	5950 3200 4900 3200
-Wire Wire Line
-	4900 3200 4900 3150
 Wire Wire Line
 	2950 2850 3000 2850
@@
 	1    0    0    -1
 $EndComp
+Wire Wire Line
+	6000 2750 5950 2750
+Wire Wire Line
+	5950 2750 5950 3200
+Wire Wire Line
+	5950 3200 4900 3200
+Wire Wire Line
+	4900 3200 4900 3150
+Wire Wire Line
+	6000 2850 5600 2850
+Wire Wire Line
+	5600 2850 5600 2450
+Wire Wire Line
+	5600 2450 4800 2450
+Wire Wire Line
+	4800 2450 4800 2550
+Wire Wire Line
+	5000 2400 5000 2550
+Wire Wire Line
+	5000 2400 5950 2400
+Wire Wire Line
+	6000 2650 5950 2650
+Wire Wire Line
+	5950 2650 5950 2400
 $EndSCHEMATC

Commit message: Added Images
Parts:
- R1, R2: value R -> 330R
- R3: value R -> 1KR
